Commit message: change package links to absolute paths

File: astrobee_dock/urdf/model.urdf (robot description, URDF)
Before this commit: robot dock, 1 links, 0 joints
Links:
- link body: geometry collision mesh filename=/home/dan/astrobee_pybullet/astrobee_media/astrobee_dock/me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; visual mesh filename=/home/dan/astrobee_pybullet/astrobee_media/astrobee_dock/me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

File: astrobee_granite/urdf/model.urdf (robot description, URDF)
Before this commit: robot granite, 1 links, 0 joints
Links:
- link body: geometry collision box size=0.01 0.9 2.0; collision box size=0.01 0.9 2.0

File: astrobee_handrail_21_5/urdf/model.urdf (robot description, URDF)
Before this commit: robot handrail, 1 links, 0 joints
Links:
- link body: geometry collision mesh filename=/home/dan/astrobee_pybullet/astrobee_media/astrobee_handrai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; visual mesh filename=/home/dan/astrobee_pybullet/astrobee_media/astrobee_handrai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

File: astrobee_handrail_30/urdf/model.urdf (robot description, URDF)
Before this commit: robot handrail, 1 links, 0 joints
Links:
- link body: geometry collision mesh filename=/home/dan/astrobee_pybullet/astrobee_media/astrobee_handrai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; visual mesh filename=/home/dan/astrobee_pybullet/astrobee_media/astrobee_handrai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

File: astrobee_handrail_41_5/urdf/model.urdf (robot description, URDF)
Before this commit: robot handrail, 1 links, 0 joints
Links:
- link body: geometry collision mesh filename=/home/dan/astrobee_pybullet/astrobee_media/astrobee_handrai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; visual mesh filename=/home/dan/astrobee_pybullet/astrobee_media/astrobee_handrai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

File: astrobee_handrail_8_5/urdf/model.urdf (robot description, URDF)
Before this commit: robot handrail, 1 links, 0 joints
Links:
- link body: geometry collision mesh filename=/home/dan/astrobee_pybullet/astrobee_media/astrobee_handrai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; visual mesh filename=/home/dan/astrobee_pybullet/astrobee_media/astrobee_handrai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

File: astrobee_iss/urdf/model.urdf (robot description, URDF)
Before this commit: robot iss, 1 links, 0 joints
Links:
- link body: geometry collision mesh filename=/home/dan/astrobee_pybullet/astrobee_media/astrobee_iss/mes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; collision mesh filename=/home/dan/astrobee_pybullet/astrobee_media/astrobee_iss/mes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
