Commit message: comment out cupola and node 1 until vhacd issue is fixed

File: astrobee_iss/urdf/model.urdf (robot description, URDF)
Before this commit: robot iss, 1 links, 0 joints
Links:
- link body: geometry collision mesh filename=/home/dan/astrobee_pybullet/astrobee_media/astrobee_iss/mes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; collision mesh filename=/home/dan/astrobee_pybullet/astrobee_media/astrobee_iss/mes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
